File: Hardware/Heat Controller.kicad_pcb (KiCad board)
At the start: 2 copper layers, 72 x 63 mm, 25 parts, among them J1 Screw_Terminal_01x03, J2 Screw_Terminal_01x03, J3 Conn_01x03_Male, J4 Conn_01x04_Male, K1 SANYOU_SRD_Form_C, Q1 BC547, SW1 SW_Push, U1 DS18B20, U2 ATtiny85-20PU

Commit message: Updated PCB according to schematic change.
Added 4K7 resistor for one-wire signal line. Updated connections to ATtiny85 to work with I2C OLED display. To be rerouted.
Parts:
- added R6: 4K7, Resistor_THT:R_Axial_DIN0207_L6.3mm_D2.5mm_P7.62mm_Horizontal, F.Cu at (187.2, 88.8)
- F2: value 0.1 A -> 0.2 A
Connections:
- U2 pad 1: /SDA -> /LEDControl
- U2 pad 2: /ButtonPin -> /Temp
- U2 pad 3: /SCL -> /RelayControl
- U2 pad 5: /LEDControl -> /SDA
- U2 pad 6: /RelayControl -> /ButtonPin
- U2 pad 7: /Temp -> /SCL
Changed lines of the file:
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@@
     (tracks 193)
     (zones 0)
-    (modules 25)
+    (modules 26)
     (nets 22)
   )
@@
       (effects (font (size 1 1) (thickness 0.15)))
     )
-    (fp_text value "0.1 A" (at -3 3 90) (layer F.Fab)
+    (fp_text value "0.2 A" (at -3 3 90) (layer F.Fab)
       (effects (font (size 1 1) (thickness 0.15)))
     )
@@
       (net 1 GND))
     (pad 7 thru_hole oval (at 7.62 2.54) (size 1.6 1.6) (drill 0.8) (layers *.Cu *.Mask)
+      (net 14 /SCL))
+    (pad 3 thru_hole oval (at 0 5.08) (size 1.6 1.6) (drill 0.8) (layers *.Cu *.Mask)
+      (net 12 /RelayControl))
+    (pad 6 thru_hole oval (at 7.62 5.08) (size 1.6 1.6) (drill 0.8) (layers *.Cu *.Mask)
+      (net 17 /ButtonPin))
+    (pad 2 thru_hole oval (at 0 2.54) (size 1.6 1.6) (drill 0.8) (layers *.Cu *.Mask)
       (net 19 /Temp))
-    (pad 3 thru_hole oval (at 0 5.08) (size 1.6 1.6) (drill 0.8) (layers *.Cu *.Mask)
-      (net 14 /SCL))
-    (pad 6 thru_hole oval (at 7.62 5.08) (size 1.6 1.6) (drill 0.8) (layers *.Cu *.Mask)
-      (net 12 /RelayControl))
-    (pad 2 thru_hole oval (at 0 2.54) (size 1.6 1.6) (drill 0.8) (layers *.Cu *.Mask)
-      (net 17 /ButtonPin))
     (pad 5 thru_hole oval (at 7.62 7.62) (size 1.6 1.6) (drill 0.8) (layers *.Cu *.Mask)
+      (net 13 /SDA))
+    (pad 1 thru_hole rect (at 0 0) (size 1.6 1.6) (drill 0.8) (layers *.Cu *.Mask)
       (net 18 /LEDControl))
-    (pad 1 thru_hole rect (at 0 0) (size 1.6 1.6) (drill 0.8) (layers *.Cu *.Mask)
-      (net 13 /SDA))
     (model ${KISYS3DMOD}/Package_DIP.3dshapes/DIP-8_W7.62mm.wrl
       (at (xyz 0 0 0))
@@
     )
   )
+  (module Resistor_THT:R_Axial_DIN0207_L6.3mm_D2.5mm_P7.62mm_Horizontal (layer F.Cu)
+    (at 187.25 88.75)
+    (descr "Resistor, Axial_DIN0207 series, Axial, Horizontal, pin pitch=7.62mm, 0.25W = 1/4W, length*diameter=6.3*2.5mm^2, http://cdn-reichelt.de/documents/datenblatt/B400/1_4W%23YAG.pdf")
+    (tags "Resistor Axial_DIN0207 series Axial Horizontal pin pitch 7.62mm 0.25W = 1/4W length 6.3mm diameter 2.5mm")
+    (fp_text reference R6 (at 3.81 -2.37) (layer F.SilkS)
+      (effects (font (size 1 1) (thickness 0.15)))
+    )
+    (fp_text value 4K7 (at 3.81 2.37) (layer F.Fab)
+      (effects (font (size 1 1) (thickness 0.15)))
+    )
+    (fp_line (start 0.66 -1.25) (end 0.66 1.25) (layer F.Fab) (width 0.1))
+    (fp_line (start 0.66 1.25) (end 6.96 1.25) (layer F.Fab) (width 0.1))
+    (fp_line (start 6.96 1.25) (end 6.96 -1.25) (layer F.Fab) (width 0.1))
+    (fp_line (start 6.96 -1.25) (end 0.66 -1.25) (layer F.Fab) (width 0.1))
+    (fp_line (start 0 0) (end 0.66 0) (layer F.Fab) (width 0.1))
+    (fp_line (start 7.62 0) (end 6.96 0) (layer F.Fab) (width 0.1))
+    (fp_line (start 0.54 -1.04) (end 0.54 -1.37) (layer F.SilkS) (width 0.12))
+    (fp_line (start 0.54 -1.37) (end 7.08 -1.37) (layer F.SilkS) (width 0.12))
+    (fp_line (start 7.08 -1.37) (end 7.08 -1.04) (layer F.SilkS) (width 0.12))
+    (fp_line (start 0.54 1.04) (end 0.54 1.37) (layer F.SilkS) (width 0.12))
+    (fp_line (start 0.54 1.37) (end 7.08 1.37) (layer F.SilkS) (width 0.12))
+    (fp_line (start 7.08 1.37) (end 7.08 1.04) (layer F.SilkS) (width 0.12))
+    (fp_line (start -1.05 -1.5) (end -1.05 1.5) (layer F.CrtYd) (width 0.05))
+    (fp_line (start -1.05 1.5) (end 8.67 1.5) (layer F.CrtYd) (width 0.05))
+    (fp_line (start 8.67 1.5) (end 8.67 -1.5) (layer F.CrtYd) (width 0.05))
+    (fp_line (start 8.67 -1.5) (end -1.05 -1.5) (layer F.CrtYd) (width 0.05))
+    (fp_text user %R (at 3.81 0) (layer F.Fab)
+      (effects (font (size 1 1) (thickness 0.15)))
+    )
+    (pad 1 thru_hole circle (at 0 0) (size 1.6 1.6) (drill 0.8) (layers *.Cu *.Mask)
+      (net 20 +5V))
+    (pad 2 thru_hole oval (at 7.62 0) (size 1.6 1.6) (drill 0.8) (layers *.Cu *.Mask)
+      (net 19 /Temp))
+    (model ${KISYS3DMOD}/Resistor_THT.3dshapes/R_Axial_DIN0207_L6.3mm_D2.5mm_P7.62mm_Horizontal.wrl
+      (at (xyz 0 0 0))
+      (scale (xyz 1 1 1))
+      (rotate (xyz 0 0 0))
+    )
+  )
   (gr_text "\"De vorst besefte het nog niet,\nmaar hij had al verloren...\"" (at 120.5 104 270) (layer B.SilkS)
     (effects (font (size 1 1) (thickness 0.15) italic) (justify mirror))
@@
   (via (at 159.25 125.75) (size 0.8) (drill 0.4) (layers F.Cu B.Cu) (net 1))
   (segment (start 155.75 125.75) (end 159.25 125.75) (width 0.25) (layer B.Cu) (net 1))
+  (via (at 158.5 120) (size 0.8) (drill 0.4) (layers F.Cu B.Cu) (net 1))
+  (segment (start 156.86 120) (end 156.845 120.015) (width 0.25) (layer F.Cu) (net 1))
+  (segment (start 158.5 120) (end 156.86 120) (width 0.25) (layer F.Cu) (net 1))
+  (via (at 161.25 123.25) (size 0.8) (drill 0.4) (layers F.Cu B.Cu) (net 1))
+  (segment (start 159.25 125.75) (end 160.5 125.75) (width 0.25) (layer B.Cu) (net 1))
+  (segment (start 160.5 125.75) (end 161.25 125) (width 0.25) (layer B.Cu) (net 1))
+  (segment (start 161.25 125) (end 161.25 123.25) (width 0.25) (layer B.Cu) (net 1))
+  (via (at 176.5 120.5) (size 0.8) (drill 0.4) (layers F.Cu B.Cu) (net 1))
+  (via (at 176.5 113) (size 0.8) (drill 0.4) (layers F.Cu B.Cu) (net 1))
+  (segment (start 176.5 113.25) (end 176.5 120.5) (width 0.25) (layer B.Cu) (net 1))
   (segment (start 150 117.4) (end 150 110.5) (width 0.25) (layer B.Cu) (net 2))
   (segment (start 156 110) (end 156.845 109.155) (width 0.25) (layer B.Cu) (net 2))
@@
   (segment (start 138.14 98.25) (end 139.75 99.86) (width 1.5) (layer F.Cu) (net 6))
   (segment (start 129.5 98.25) (end 138.14 98.25) (width 1.5) (layer F.Cu) (net 6))
-  (segment (start 171.45 78.74141) (end 171.45 78.740705) (width 0.25) (layer B.Cu) (net 20))
   (segment (start 145.35 91.75) (end 139.7 86.1) (width 1.5) (layer F.Cu) (net 7))
   (segment (start 148 91.75) (end 145.35 91.75) (width 1.5) (layer F.Cu) (net 7))
@@
   (segment (start 163 113.5) (end 163 111.5) (width 0.25) (layer F.Cu) (net 19))
   (segment (start 163 111.5) (end 163.5 111) (width 0.25) (layer F.Cu) (net 19))
+  (segment (start 171.45 78.74141) (end 171.45 78.740705) (width 0.25) (layer B.Cu) (net 20))
   (via (at 167.5 120.75) (size 0.8) (drill 0.4) (layers F.Cu B.Cu) (net 20))
   (segment (start 167.5 118.885) (end 167.64 118.745) (width 0.25) (layer F.Cu) (net 20))
@@
   (segment (start 166 118.205) (end 166.54 118.745) (width 0.25) (layer F.Cu) (net 20))
   (segment (start 166 113.93) (end 166 118.205) (width 0.25) (layer F.Cu) (net 20))
-  (via (at 158.5 120) (size 0.8) (drill 0.4) (layers F.Cu B.Cu) (net 1))
-  (segment (start 156.86 120) (end 156.845 120.015) (width 0.25) (layer F.Cu) (net 1))
-  (segment (start 158.5 120) (end 156.86 120) (width 0.25) (layer F.Cu) (net 1))
-  (via (at 161.25 123.25) (size 0.8) (drill 0.4) (layers F.Cu B.Cu) (net 1))
-  (segment (start 159.25 125.75) (end 160.5 125.75) (width 0.25) (layer B.Cu) (net 1))
-  (segment (start 160.5 125.75) (end 161.25 125) (width 0.25) (layer B.Cu) (net 1))
-  (segment (start 161.25 125) (end 161.25 123.25) (width 0.25) (layer B.Cu) (net 1))
-  (via (at 176.5 120.5) (size 0.8) (drill 0.4) (layers F.Cu B.Cu) (net 1))
-  (via (at 176.5 113) (size 0.8) (drill 0.4) (layers F.Cu B.Cu) (net 1))
-  (segment (start 176.5 113.25) (end 176.5 120.5) (width 0.25) (layer B.Cu) (net 1))
   (segment (start 120.65 104.14) (end 120.65 87.1) (width 1.5) (layer F.Cu) (net 21))
   (segment (start 129.5 109.75) (end 126.26 109.75) (width 1.5) (layer F.Cu) (net 21))
