File: Hardware/Heat Controller.kicad_pcb (KiCad board)
At the start: 2 copper layers, 72 x 63 mm, 26 parts, among them J1 Screw_Terminal_01x03, J2 Screw_Terminal_01x03, J3 Conn_01x03_Male, J4 Conn_01x04_Male, K1 SANYOU_SRD_Form_C, Q1 BC547, SW1 SW_Push, U1 DS18B20, U2 ATtiny85-20PU

Commit message: Test vias for ADCD converter
Routing:
- net GND: vias 6 -> 7
- net +5V: vias 2 -> 3
Other:
- board text added: "5V-GND"
Changed lines of the file:
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@@
   (general
     (thickness 1.6)
-    (drawings 23)
-    (tracks 193)
+    (drawings 24)
+    (tracks 195)
     (zones 0)
     (modules 26)
@@
     )
   )
+  (gr_text 5V-GND (at 178.25 106) (layer F.SilkS)
+    (effects (font (size 0.5 0.5) (thickness 0.125)))
+  )
   (gr_line (start 108.25 72.5) (end 180 72.5) (layer Edge.Cuts) (width 0.05))
   (gr_line (start 108.25 135.5) (end 108.25 72.5) (layer Edge.Cuts) (width 0.05))
@@
   (via (at 176.5 113) (size 0.8) (drill 0.4) (layers F.Cu B.Cu) (net 1))
   (segment (start 176.5 113.25) (end 176.5 120.5) (width 0.25) (layer B.Cu) (net 1))
+  (via (at 179 105.25) (size 0.8) (drill 0.4) (layers F.Cu B.Cu) (net 1))
   (segment (start 150 117.4) (end 150 110.5) (width 0.25) (layer B.Cu) (net 2))
   (segment (start 156 110) (end 156.845 109.155) (width 0.25) (layer B.Cu) (net 2))
@@
   (segment (start 166 118.205) (end 166.54 118.745) (width 0.25) (layer F.Cu) (net 20))
   (segment (start 166 113.93) (end 166 118.205) (width 0.25) (layer F.Cu) (net 20))
+  (via (at 177.25 105.25) (size 0.8) (drill 0.4) (layers F.Cu B.Cu) (net 20))
   (segment (start 120.65 104.14) (end 120.65 87.1) (width 1.5) (layer F.Cu) (net 21))
   (segment (start 129.5 109.75) (end 126.26 109.75) (width 1.5) (layer F.Cu) (net 21))

Commit message: Prepared PCB for ordering
Parts:
- removed J3: Conn_01x03_Male, Connector_PinHeader_2.54mm:PinHeader_1x03_P2.54mm_Vertical
- added H4: MountingHole, MountingHole:MountingHole_4.5mm, F.Cu at (138.8, 128.5)
- added JP1: Jumper_3_Open, Connector_PinHeader_2.54mm:PinHeader_1x03_P2.54mm_Vertical, F.Cu at (168.0, 113.8)
- R2: value 10K -> 150
- R3, R4, R5: value 220 -> 360
- moved R6 48.8 mm to (164.2, 131.8), turned to 90 degrees
- moved D1 8.25 mm to (145.8, 133.2)
- moved J4 7.58 mm to (171.5, 132.0), turned to 180 degrees
- moved R1 6.75 mm to (149.2, 131.8)
- moved R5 6.25 mm to (152.2, 131.8)
- moved R4 6.00 mm to (155.2, 131.8)
- moved R3 5.75 mm to (158.2, 131.8)
- moved R2 5.50 mm to (161.2, 124.1)
- moved U2 0.41 mm to (157.2, 112.4)
- moved SW1 0.38 mm to (175.0, 116.8)
Connections:
- net /SCL renamed SCL
- net /SDA renamed SDA
- net /Temp renamed TempPin
- D3 pad 1: GND -> Net-(D3-Pad1)
- D3 pad 2: Net-(D3-Pad2) -> +5V
- R2 pad 1: GND -> Net-(R2-Pad1)
- R2 pad 2: /ButtonPin -> ControlPin
- R4 pad 1: Net-(D3-Pad2) -> ControlPin
- R4 pad 2: /LEDControl -> Net-(D3-Pad1)
- R5 pad 2: /RelayControl -> RelayPin
- SW1 pad 1: +5V -> Net-(R2-Pad1)
- SW1 pad 2: /ButtonPin -> GND
- U2 pad 1: /LEDControl -> Net-(U2-Pad1)
- U2 pad 3: /RelayControl -> ControlPin
- U2 pad 6: /ButtonPin -> RelayPin
Routing:
- net Net-(D3-Pad1): track 0.00 -> 50.7 mm
- net /ButtonPin: track 50.2 -> 0.00 mm, vias 1 -> 0
- net /RelayControl: track 38.1 -> 0.00 mm
- net Net-(D3-Pad2): track 31.3 -> 0.00 mm
- net RelayPin: track 0.00 -> 23.7 mm
- net Net-(R2-Pad1): track 0.00 -> 22.6 mm, vias 0 -> 1
- net ControlPin: track 0.00 -> 22.1 mm
- net +5V: track 27.8 -> 9.95 mm, vias 3 -> 7
- net TempPin: track 20.6 -> 38.0 mm
- net /LEDControl: track 16.9 -> 0.00 mm, vias 1 -> 0
- net SDA: track 24.7 -> 15.5 mm
- net Net-(JP1-Pad2): track 40.3 -> 32.0 mm, vias 0 -> 2
- net Net-(D4-Pad2): track 31.5 -> 26.9 mm
- net SCL: track 20.8 -> 17.3 mm
- net Net-(D2-Pad2): track 32.5 -> 29.1 mm
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Other:
- board size 72 x 63 mm -> 72.5 x 63 mm
- board text added: "INPUT (1: Earth - 2: N - 3: L) OUTPUT"
- board text removed: "1: Earth - 2: N - 3: L"
