File: Hardware/Heat Controller.sch (KiCad schematic (older format))
At the start: 26 parts, among them J1 Screw_Terminal_01x03, J2 Screw_Terminal_01x03, J3 Conn_01x03_Male, J4 Conn_01x04_Male, K1 SANYOU_SRD_Form_C, Q1 BC547, SW1 SW_Push, U1 DS18B20, U2 ATtiny85-20PU

Commit message: Remplaced normal terminal for jumper
Parts:
- removed J3: Conn_01x03_Male, Connector_PinHeader_2.54mm:PinHeader_1x03_P2.54mm_Vertical, symbol Connector:Conn_01x03_Male
- added JP1: Jumper_3_Open, Connector_PinHeader_2.54mm:PinHeader_1x03_P2.54mm_Vertical, symbol Jumper:Jumper_3_Open
Connections:
- net +5V: now also JP1.3 (B)
- net RelayControl: now also JP1.1 (A)
- net at R1.1: now also JP1.2 (C)
Other:
- note added: "Input (from grid):\n3 - L\n2 - N\n1 - Earth"
- note added: "Jumper allows to pick between:\n-always off (no header attached)\n-always on (header to comm and +5V)\n-controlled (header to comm and relaycontrol)"
- note added: "Output (to heater):\n3 - L (switched)\n2 - N\n1 - Earth"
- note removed: "Header allows to pick between:\n-always off (no header attached)\n-always on (header to comm and +5V)\n-controlled (header to comm and relaycontrol)"
- note removed: "Input (from grid):\n3 - L\n2 - N\n1 - GND"
- note removed: "Output (to heater):\n3 - L (switched)\n2 - N\n1 - GND"
Changed lines of the file:
@@
 	2500 3650 2500 3400
 Text Notes 600  2700 0    50   ~ 0
-Input (from grid):\n3 - L\n2 - N\n1 - GND
+Input (from grid):\n3 - L\n2 - N\n1 - Earth
 Text Notes 600  3650 0    50   ~ 0
-Output (to heater):\n3 - L (switched)\n2 - N\n1 - GND
+Output (to heater):\n3 - L (switched)\n2 - N\n1 - Earth
 Wire Wire Line
 	8800 850  9000 850
@@
 	2400 2550 2400 3500
 Connection ~ 2400 2550
-Text Label 5400 3650 0    50   ~ 0
-RelayControl
 Wire Wire Line
 	4450 4150 4450 4350
@@
 	8300 4300 9200 4300
 Wire Wire Line
-	5400 3650 5400 3850
-Wire Wire Line
-	5400 4050 5400 4300
-Wire Wire Line
 	8000 1550 8500 1550
 Wire Wire Line
@@
 Text Label 10050 3450 0    50   ~ 0
 ButtonPin
-$Comp
-L Connector:Conn_01x03_Male J3
-U 1 1 5F739462
-P 5800 3950
-F 0 "J3" H 5772 3882 50  0000 R CNN
-F 1 "Conn_01x03_Male" H 5772 3973 50  0000 R CNN
-F 2 "Connector_PinHeader_2.54mm:PinHeader_1x03_P2.54mm_Vertical" H 5800 3950 50  0001 C CNN
-F 3 "~" H 5800 3950 50  0001 C CNN
-	1    5800 3950
-	-1   0    0    1
-$EndComp
-Wire Wire Line
-	5400 3850 5600 3850
 Wire Wire Line
 	5250 3950 5600 3950
-Wire Wire Line
-	5400 4050 5600 4050
 $Comp
 L power:GND #PWR07
@@
 Wire Wire Line
 	5700 5400 5700 5350
-$Comp
-L power:+5V #PWR05
-U 1 1 5F7C8495
-P 5300 4300
-F 0 "#PWR05" H 5300 4150 50  0001 C CNN
-F 1 "+5V" H 5315 4473 50  0000 C CNN
-F 2 "" H 5300 4300 50  0001 C CNN
-F 3 "" H 5300 4300 50  0001 C CNN
-	1    5300 4300
-	1    0    0    -1
-$EndComp
-Wire Wire Line
-	5300 4300 5400 4300
 Wire Notes Line
 	3350 1900 3350 4100
@@
 Power input and control section.\nVAC comes in through screw terminal and feeds the ACDC converter.\nSecondly, the L is switched through a relay.\nTwo grounded mounting holes are added, as they are located close to the terminals.
 Text Notes 4700 4900 0    50   ~ 0
-Header allows to pick between:\n-always off (no header attached)\n-always on (header to comm and +5V)\n-controlled (header to comm and relaycontrol)
+Jumper allows to pick between:\n-always off (no header attached)\n-always on (header to comm and +5V)\n-controlled (header to comm and relaycontrol)
 Wire Wire Line
 	4450 3750 4450 3650
@@
 Wire Wire Line
 	5700 5350 5700 5250
+$Comp
+L Jumper:Jumper_3_Open JP1
+U 1 1 5F83BB74
+P 5750 3950
+F 0 "JP1" V 5704 4037 50  0000 L CNN
+F 1 "Jumper_3_Open" V 5795 4037 50  0000 L CNN
+F 2 "Connector_PinHeader_2.54mm:PinHeader_1x03_P2.54mm_Vertical" H 5750 3950 50  0001 C CNN
+F 3 "~" H 5750 3950 50  0001 C CNN
+	1    5750 3950
+	0    1    1    0
+$EndComp
+Text Label 5750 3600 0    50   ~ 0
+RelayControl
+$Comp
+L power:+5V #PWR05
+U 1 1 5F7C8495
+P 5750 4300
+F 0 "#PWR05" H 5750 4150 50  0001 C CNN
+F 1 "+5V" H 5765 4473 50  0000 C CNN
+F 2 "" H 5750 4300 50  0001 C CNN
+F 3 "" H 5750 4300 50  0001 C CNN
+	1    5750 4300
+	-1   0    0    1
+$EndComp
+Wire Wire Line
+	5750 3700 5750 3600
+Wire Wire Line
+	5750 4300 5750 4200
 $EndSCHEMATC

Commit message: Prepared PCB for ordering
Parts:
- added H4: MountingHole, MountingHole:MountingHole_4.5mm, symbol Mechanical:MountingHole
- R2: value 10K -> 150
- R3, R4, R5: value 220 -> 360
Connections:
- net +5V: now also D3.2 (A); no longer SW1.1
- net GND: now also SW1.2; no longer D3.1 (K), R2.1
- net ControlPin: now reaches R4.1
- net ControlPin: now also R2.2, U2.3 (XTAL2/PB4); no longer D3.2 (A)
- removed net ButtonPin: R2.2, SW1.2, U2.6 (PB1)
- net LEDControl: no longer names the net of U2.1 (~RESET~/PB5)
- net LEDControl: no longer R4.2
- net RelayControl renamed RelayPin
- net RelayPin: now also U2.6 (PB1); no longer U2.3 (XTAL2/PB4)
- net Temp renamed TempPin
- new net: D3.1 (K), R4.2
- new net: R2.1, SW1.1
- no-connect marks 1 -> 2
Other:
- note added: "Jumper allows to pick between:\n-always off (no header attached)\n-always on (header to comm and +5V)\n-controlled (header to comm and relaypin)"
- note added: "Status LED's:\n- green1: power indicator\n- red: relay indicator\n- green2: control indicator (combined with button on 1 pin)"
- note removed: "Control button"
- note removed: "Jumper allows to pick between:\n-always off (no header attached)\n-always on (header to comm and +5V)\n-controlled (header to comm and relaycontrol)"
- note removed: "Status LED's:\n- green: power indicator\n- green: control indicator\n- red: relay indicator"
- moved on the sheet: D2, D3, D4, R2, R3, R4, R5, R6, SW1, U1
